File: V1/IRL540_HBridge_V1/IRL540_HBridge_V1.sch (KiCad schematic (older format))
At the start: 16 parts, among them IC1 7400, IC2 7408, J1 CTRL, Q1 IRL540N, Q2 IRL540N, Q3 IRL540N, Q4 IRL540N

Commit message: Enrutado y silks
Parts:
- removed J1: CTRL, Connector_PinHeader_1.27mm:PinHeader_2x05_P1.27mm_Vertical, symbol Connector_Generic:Conn_02x05_Counter_Clockwise
- added J1: Conn_01x05_Male, Connector_PinHeader_2.54mm:PinHeader_1x05_P2.54mm_Vertical, symbol Connector:Conn_01x05_Male
- added J2: Conn_01x02_Male, Connector_PinHeader_2.54mm:PinHeader_1x02_P2.54mm_Vertical, symbol Connector:Conn_01x02_Male
- added LED1: LED, LED_THT:LED_D3.0mm, symbol Device:LED
- added R4: 220, Resistor_THT:R_Axial_DIN0204_L3.6mm_D1.6mm_P5.08mm_Horizontal, symbol Device:R
Connections:
- net +5V: now also J1.1 (Pin_1), J2.1 (Pin_1), J2.2 (Pin_2), LED1.2 (A)
- net EN: now also J1.2 (Pin_2)
- net GNDREF: now also J1.5 (Pin_5), R4.2
- net I_A: now also J1.3 (Pin_3)
- net I_B: now also J1.4 (Pin_4)
- new net: LED1.1 (K), R4.1
Other:
- moved on the sheet: BAT1
Changed lines of the file:
@@
 	8250 4450 8250 4650
-$Comp
-L Connector_Generic:Conn_02x05_Counter_Clockwise J1
-U 1 1 621E8254
-P 2750 5850
-F 0 "J1" H 2800 6267 50  0001 C CNN
-F 1 "CTRL" H 2800 6175 50  0000 C CNN
-F 2 "Connector_PinHeader_1.27mm:PinHeader_2x05_P1.27mm_Vertical" H 2750 5850 50  0001 C CNN
-F 3 "~" H 2750 5850 50  0001 C CNN
-	1    2750 5850
-	1    0    0    -1
-$EndComp
 $Comp
 L power:GNDREF #PWR0110
 U 1 1 621EB6B1
-P 2350 5650
-F 0 "#PWR0110" H 2350 5400 50  0001 C CNN
-F 1 "GNDREF" H 2355 5477 50  0001 C CNN
-F 2 "" H 2350 5650 50  0001 C CNN
-F 3 "" H 2350 5650 50  0001 C CNN
-	1    2350 5650
-	0    1    1    0
+P 2550 6200
+F 0 "#PWR0110" H 2550 5950 50  0001 C CNN
+F 1 "GNDREF" H 2555 6027 50  0001 C CNN
+F 2 "" H 2550 6200 50  0001 C CNN
+F 3 "" H 2550 6200 50  0001 C CNN
+	1    2550 6200
+	1    0    0    -1
 $EndComp
 $Comp
@@
 Text GLabel 1750 5950 0    50   Output ~ 0
 I_A
-Wire Wire Line
-	2350 5650 2550 5650
-Wire Wire Line
-	2350 5750 2550 5750
-Wire Wire Line
-	2550 5750 3050 5750
-Connection ~ 2550 5750
-Wire Wire Line
-	3050 5850 3050 5750
-Connection ~ 3050 5750
 $Comp
 L Connector_Generic:Conn_01x02 MOT1
@@
 L Connector_Generic:Conn_01x02 BAT1
 U 1 1 621E096C
-P 3900 6050
-F 0 "BAT1" V 3772 6130 50  0000 L CNN
-F 1 "Conn_01x02" V 3863 6130 50  0000 L CNN
-F 2 "Connector:JWT_A3963_1x02_P3.96mm_Vertical" H 3900 6050 50  0001 C CNN
-F 3 "~" H 3900 6050 50  0001 C CNN
-	1    3900 6050
+P 4200 6750
+F 0 "BAT1" V 4072 6830 50  0000 L CNN
+F 1 "Conn_01x02" V 4163 6830 50  0000 L CNN
+F 2 "Connector:JWT_A3963_1x02_P3.96mm_Vertical" H 4200 6750 50  0001 C CNN
+F 3 "~" H 4200 6750 50  0001 C CNN
+	1    4200 6750
 	0    1    1    0
 $EndComp
@@
 L power:VDD #PWR0112
 U 1 1 621E1EBC
-P 3800 5650
-F 0 "#PWR0112" H 3800 5500 50  0001 C CNN
-F 1 "VDD" H 3815 5823 50  0000 C CNN
-F 2 "" H 3800 5650 50  0001 C CNN
-F 3 "" H 3800 5650 50  0001 C CNN
-	1    3800 5650
+P 4100 6350
+F 0 "#PWR0112" H 4100 6200 50  0001 C CNN
+F 1 "VDD" H 4115 6523 50  0000 C CNN
+F 2 "" H 4100 6350 50  0001 C CNN
+F 3 "" H 4100 6350 50  0001 C CNN
+	1    4100 6350
 	1    0    0    -1
 $EndComp
@@
 L power:GNDREF #PWR0113
 U 1 1 621E4DED
-P 3900 5650
-F 0 "#PWR0113" H 3900 5400 50  0001 C CNN
-F 1 "GNDREF" H 3905 5477 50  0001 C CNN
-F 2 "" H 3900 5650 50  0001 C CNN
-F 3 "" H 3900 5650 50  0001 C CNN
-	1    3900 5650
+P 4200 6350
+F 0 "#PWR0113" H 4200 6100 50  0001 C CNN
+F 1 "GNDREF" H 4205 6177 50  0001 C CNN
+F 2 "" H 4200 6350 50  0001 C CNN
+F 3 "" H 4200 6350 50  0001 C CNN
+	1    4200 6350
 	-1   0    0    1
 $EndComp
 Wire Wire Line
-	3900 5650 3900 5850
-Wire Wire Line
-	3800 5650 3800 5850
+	4200 6350 4200 6550
+Wire Wire Line
+	4100 6350 4100 6550
 $Comp
 L 74xx_dip_14:74XX_DIP_14 IC1
@@
 	1    0    0    -1
 $EndComp
+$Comp
+L Connector:Conn_01x05_Male J1
+U 1 1 621BDE75
+P 2750 5950
+F 0 "J1" H 2722 5974 50  0000 R CNN
+F 1 "Conn_01x05_Male" H 2722 5883 50  0000 R CNN
+F 2 "Connector_PinHeader_2.54mm:PinHeader_1x05_P2.54mm_Vertical" H 2750 5950 50  0001 C CNN
+F 3 "~" H 2750 5950 50  0001 C CNN
+	1    2750 5950
+	-1   0    0    -1
+$EndComp
+$Comp
+L Connector:Conn_01x02_Male J2
+U 1 1 621C222B
+P 2900 5750
+F 0 "J2" H 3008 5931 50  0000 C CNN
+F 1 "Conn_01x02_Male" H 3008 5840 50  0000 C CNN
+F 2 "Connector_PinHeader_2.54mm:PinHeader_1x02_P2.54mm_Vertical" H 2900 5750 50  0001 C CNN
+F 3 "~" H 2900 5750 50  0001 C CNN
+	1    2900 5750
+	1    0    0    -1
+$EndComp
+Wire Wire Line
+	2550 5750 2350 5750
+Wire Wire Line
+	3100 5750 2550 5750
+Wire Wire Line
+	3100 5750 3100 5650
+Connection ~ 3100 5750
+Connection ~ 2550 5750
+Wire Wire Line
+	2550 6150 2550 6200
+Wire Wire Line
+	3100 5750 3100 5850
+$Comp
+L Device:LED LED1
+U 1 1 621C1E93
+P 3650 6500
+F 0 "LED1" V 3689 6382 50  0000 R CNN
+F 1 "LED" V 3598 6382 50  0000 R CNN
+F 2 "LED_THT:LED_D3.0mm" H 3650 6500 50  0001 C CNN
+F 3 "~" H 3650 6500 50  0001 C CNN
+	1    3650 6500
+	0    -1   -1   0
+$EndComp
+$Comp
+L Device:R R4
+U 1 1 621C3C99
+P 3650 6800
+F 0 "R4" H 3720 6846 50  0000 L CNN
+F 1 "220" H 3720 6755 50  0000 L CNN
+F 2 "Resistor_THT:R_Axial_DIN0204_L3.6mm_D1.6mm_P5.08mm_Horizontal" V 3580 6800 50  0001 C CNN
+F 3 "~" H 3650 6800 50  0001 C CNN
+	1    3650 6800
+	1    0    0    -1
+$EndComp
+$Comp
+L power:+5V #PWR0101
+U 1 1 621CA8BB
+P 3650 6350
+F 0 "#PWR0101" H 3650 6200 50  0001 C CNN
+F 1 "+5V" H 3665 6523 50  0000 C CNN
+F 2 "" H 3650 6350 50  0001 C CNN
+F 3 "" H 3650 6350 50  0001 C CNN
+	1    3650 6350
+	1    0    0    -1
+$EndComp
+$Comp
+L power:GNDREF #GND0103
+U 1 1 621E000C
+P 3650 6950
+F 0 "#GND0103" H 3650 6700 50  0001 C CNN
+F 1 "GNDREF" H 3655 6777 50  0001 C CNN
+F 2 "" H 3650 6950 50  0001 C CNN
+F 3 "" H 3650 6950 50  0001 C CNN
+	1    3650 6950
+	1    0    0    -1
+$EndComp
