File: V1/IRL540_HBridge_V1/IRL540_HBridge_V1.kicad_pcb (KiCad board)
At the start: 2 copper layers, 88.9 x 63.5 mm, 16 parts, among them IC1 7400, IC2 7408, J1 CTRL, Q1 IRL540N, Q2 IRL540N, Q3 IRL540N, Q4 IRL540N

Commit message: Enrutado y silks
Parts:
- added 220: 220, Resistor_THT:R_Axial_DIN0204_L3.6mm_D1.6mm_P5.08mm_Horizontal, F.Cu at (100.3, 104.1)
- added G***: LOGO, Reset:Reset, F.Cu at (121.9, 74.3)
- added J2: Conn_01x02_Male, Connector_PinHeader_2.54mm:PinHeader_1x02_P2.54mm_Vertical, F.Cu at (96.5, 100.3)
- added LED: LED, LED_THT:LED_D3.0mm, F.Cu at (104.1, 100.3)
- J1: value CTRL -> Conn_01x05_Male; footprint Connector_PinHeader_1.27mm:PinHeader_2x05_P1.27mm_Vertical -> Connector_PinHeader_2.54mm:PinHeader_1x05_P2.54mm_Vertical
- moved J1 6.48 mm to (94.0, 100.3), turned to 0 degrees
- renumbered R3 to 10k, R2 to 10k, R1 to 10k, IC1 to 7400, IC2 to 7408, BAT1 to BAT, MOT1 to MOT
Connections:
- J1 pad 1: GNDREF -> +5V
- J1 pad 2: +5V -> EN
- J1 pad 3: EN -> I_A
- J1 pad 4: I_A -> I_B
- J1 pad 5: I_B -> GNDREF
Routing:
- net GNDREF: track 0.00 -> 147.9 mm
- net VDD: track 0.00 -> 140.6 mm
- net S_A1: track 0.00 -> 77.3 mm
- net I_B: track 0.00 -> 75.4 mm
- net I_A: track 0.00 -> 74.9 mm
- net S_A2: track 0.00 -> 71.7 mm
- net EN: track 0.00 -> 65.0 mm
- net +5V: track 0.00 -> 51.2 mm
- net Net-(MOT1-Pad2): track 0.00 -> 46.5 mm
- net Net-(MOT1-Pad1): track 0.00 -> 42.7 mm
- net S_B2: track 0.00 -> 29.7 mm
- net S_B1: track 0.00 -> 27.2 mm
- net *I_B: track 0.00 -> 22.6 mm
- net *I_A: track 0.00 -> 15.0 mm
- net Net-(LED1-Pad1): track 0.00 -> 5.39 mm
Other:
- outline, holes or cut-outs redrawn
- board text added: "12V"
- board text added: "5V"
- board text added: "AE RESET"
- board text added: "EN"
- board text added: "GND"
- board text added: "IA"
- board text added: "IB"
- board text added: "IRL540_HBridge"
- board text added: "OA"
- board text added: "OB"
- board text added: "V1.0 - Jabax 2022"

Commit message: Versión 1.0!
Parts:
- renumbered BAT to BAT1, 7400 to IC1, 7408 to IC2, LED to LED1, MOT to MOT1, 10k to R1, 10k to R2, 10k to R3, 220 to R4
Routing:
- net *I_B: track 22.6 -> 46.6 mm
- net S_A1: track 77.3 -> 93.9 mm
- net EN: track 65.0 -> 77.5 mm
- net I_B: track 75.4 -> 79.0 mm
- net S_A2: track 71.7 -> 68.3 mm
- net I_A: track 74.9 -> 73.4 mm
- added copper zone on B.Cu, net GNDREF
- added copper zone on F.Cu, net GNDREF
Other:
- net class Gate Mosfet added: clearance 0.2, trace_width 1, via_dia 0.8, via_drill 0.4
